File: ASIC.kicad_sch (KiCad schematic)
At the start: 77 parts, among them U4001 MCP1824T-1202E/OT, U4002 25MHz, U4003 BM1370_mode1, U4004 MCP1824T-0802E, U4005 SN74AVC4T774, U4006 BM1370_mode1

Commit message: started to piece in the BZM2 into schematic
Parts:
- removed C4001, C4002, C4003, C4004, C4005, C4006, C4007, C4008, C4011, C4012, C4013, C4015, C4016, C4018, C4020, C4021, C4023, C4025, C4026, C4027, C4028, C4029, C4031, C4033, C4034, C4036, C4038, C4040: 1uF, Capacitor_SMD:C_0402_1005Metric, symbol Device:C_Small
- removed C4009, C4024, C4037: 0.1uF, Capacitor_SMD:C_0402_1005Metric, symbol Device:C_Small
- removed C4010, C4014, C4017, C4019, C4022, C4030, C4032, C4035, C4039, C4041: 10uF, Capacitor_SMD:C_0603_1608Metric, symbol Device:C_Small
- removed R4001: 10k, Resistor_SMD:R_0402_1005Metric, symbol Device:R_Small_US
- removed R4002, R4004: 1k, Resistor_SMD:R_0402_1005Metric, symbol Device:R_Small_US
- removed R4003: 2k, Resistor_SMD:R_0402_1005Metric, symbol Device:R_Small_US
- removed TP4001, TP4007: ROSC, bitaxe:TestPoint_Pad_1.0x0.4mm, symbol Connector:TestPoint
- removed TP4002, TP4008: LITE, bitaxe:TestPoint_Pad_1.0x0.4mm, symbol Connector:TestPoint
- removed TP4003, TP4017: INV, bitaxe:TestPoint_Pad_1.0x0.4mm, symbol Connector:TestPoint
- removed TP4006: 0V8, bitaxe:TestPoint_Pad_D1.0mm, symbol Connector:TestPoint
- removed TP4009, TP4021: RST, bitaxe:TestPoint_Pad_1.0x0.4mm, symbol Connector:TestPoint
- removed TP4010: CI, bitaxe:TestPoint_Pad_1.0x0.4mm, symbol Connector:TestPoint
- removed TP4011: RO, bitaxe:TestPoint_Pad_1.0x0.4mm, symbol Connector:TestPoint
- removed TP4012, TP4024: CLK, bitaxe:TestPoint_Pad_1.0x0.4mm, symbol Connector:TestPoint
- removed TP4013: BI, bitaxe:TestPoint_Pad_1.0x0.4mm, symbol Connector:TestPoint
- removed TP4014, TP4018: RST, bitaxe:TestPoint_Pad_D1.0mm, symbol Connector:TestPoint
- removed TP4015, TP4019: TX, bitaxe:TestPoint_Pad_D1.0mm, symbol Connector:TestPoint
- removed TP4016, TP4020: RX, bitaxe:TestPoint_Pad_D1.0mm, symbol Connector:TestPoint
- removed TP4022: CO, bitaxe:TestPoint_Pad_1.0x0.4mm, symbol Connector:TestPoint
- removed TP4023: RI, bitaxe:TestPoint_Pad_1.0x0.4mm, symbol Connector:TestPoint
- removed TP4025: BO, bitaxe:TestPoint_Pad_1.0x0.4mm, symbol Connector:TestPoint
- removed U4003, U4006: BM1370_mode1, bitaxe:BM1370, symbol bitaxe:BM1370_mode1
- removed U4004: MCP1824T-0802E, Package_TO_SOT_SMD:SOT-23-5, symbol bitaxe:MCP1824
- added A1, A5: BZM2_MODE1, bitaxe:bzm2, symbol bitaxe:BZM2_mode1
- added A4, A8: BZM2_MODE0, bitaxe:bzm2, symbol bitaxe:BZM2_mode0
- added C46, C47, C48: 0.1uF, Capacitor_SMD:C_0402_1005Metric, symbol Device:C_Small
- added C49, C50, C51, C52: 120pF, Capacitor_SMD:C_0402_1005Metric, symbol Device:C_Small
- added C57, C58, C59, C60, C61, C62, C63, C64: 1uF, Capacitor_SMD:C_0402_1005Metric, symbol Device:C_Small
- added TP15, TP16, TP17, TP18: CLKI, TestPoint:TestPoint_Pad_D1.0mm, symbol Connector:TestPoint
- added TP19, TP20, TP21: 1V2, TestPoint:TestPoint_Pad_D1.5mm, symbol Connector:TestPoint
- added U10, U8, U9: MCP1824T-1202E/OT, Package_TO_SOT_SMD:SOT-23-5, symbol bitaxe:MCP1824
- TP14: renamed from TP4005; footprint bitaxe:TestPoint_Pad_D1.0mm -> TestPoint:TestPoint_Pad_D1.0mm
- TP22: renamed from TP4004; footprint bitaxe:TestPoint_Pad_D1.0mm -> TestPoint:TestPoint_Pad_D1.5mm; now in the parts list
- U6: renamed from U4002; DK 5852-SX3M25.000E20F30THNTR-ND -> (none)
- renumbered R4005 to R28, U4001 to U11, U4005 to U7
Connections:
- net 1V2: now also A1.30 (VDDIO), C46.1, C47.1, C64.2
- net 3V3: now also C48.1
- net 5V: now also C57.2, C58.2, C59.2, C60.2, U10.1 (VIN), U10.3 (EN), U8.1 (VIN), U8.3 (EN), U9.1 (VIN), U9.3 (EN)
- net CLKI: now also A1.29 (REFCLKIN)
- net GND: now also A1.14 (VSS), A1.21 (VSS), A1.22 (VSS), A1.23 (VSS), A1.24 (VSS), A1.25 (VSS), A1.26 (VSS), A1.27 (VSS), A1.28 (VSS), A1.35 (VSS), A1.43 (VSS), A1.44 (VSS), A1.45 (VSS), A1.46 (VSS), A1.47 (VSS), A1.48 (VSS), A1.53 (VSS), A1.54 (VSS), A1.55 (VSS), A1.56 (VSS), A1.57 (VSS), A1.58 (VSS), C46.2, C47.2, C48.2, C60.1, C64.1; no longer U7.6 (A4)
- net RST_1V2: now also A1.33 (RESET_IN)
- net RX_1V2: now also A1.34 (RX_IN)
- net TX_1V2: now also A1.32 (TX_OUT)
- net TT_3V3: now reaches U7.11 (B4)
- new net: A8.38 (REFCLKOUT1), C49.1
- new net: A4.20 (REFCLKOUT2), C52.1
- new net: A4.38 (REFCLKOUT1), C50.1
- new net: A8.34 (TRIP_IN), TP18.1
- new net: A8.20 (REFCLKOUT2), C51.1
- new net: A8.31 (RX_OUT), TP15.1
- new net: A8.32 (RESET_OUT), TP16.1
- new net: A8.33 (TX_IN), TP17.1
- new net 1V2-1: A4.30 (VDDIO), C63.2, TP21.1, U10.5 (VOUT)
- new net 1V2-2: A5.30 (VDDIO), C62.2, TP20.1, U9.5 (VOUT)
- new net 1V2-3: A8.30 (VDDIO), C61.2, TP19.1, U8.5 (VOUT)
- new net GND1: A1.2 (VDD), A1.3 (VDD), A1.4 (VDD), A1.41 (VDD), A1.42 (VDD), A1.49 (VDD), A1.5 (VDD), A1.50 (VDD), A1.51 (VDD), A1.52 (VDD), A1.59 (VDD), A1.6 (VDD), A1.60 (VDD), A1.7 (VDD), A1.8 (VDD), A4.14 (VSS), A4.21 (VSS), A4.22 (VSS), A4.23 (VSS), A4.24 (VSS), A4.25 (VSS), A4.26 (VSS), A4.27 (VSS), A4.28 (VSS), A4.35 (VSS), A4.36 (PINSEL), A4.43 (VSS), A4.44 (VSS), A4.45 (VSS), A4.46 (VSS), A4.47 (VSS), A4.48 (VSS), A4.53 (VSS), A4.54 (VSS), A4.55 (VSS), A4.56 (VSS), A4.57 (VSS), A4.58 (VSS), C50.2, C52.2, C59.1, C63.1, U10.2 (GND)
- new net GND2: A4.2 (VDD), A4.3 (VDD), A4.4 (VDD), A4.41 (VDD), A4.42 (VDD), A4.49 (VDD), A4.5 (VDD), A4.50 (VDD), A4.51 (VDD), A4.52 (VDD), A4.59 (VDD), A4.6 (VDD), A4.60 (VDD), A4.7 (VDD), A4.8 (VDD), A5.14 (VSS), A5.21 (VSS), A5.22 (VSS), A5.23 (VSS), A5.24 (VSS), A5.25 (VSS), A5.26 (VSS), A5.27 (VSS), A5.28 (VSS), A5.35 (VSS), A5.43 (VSS), A5.44 (VSS), A5.45 (VSS), A5.46 (VSS), A5.47 (VSS), A5.48 (VSS), A5.53 (VSS), A5.54 (VSS), A5.55 (VSS), A5.56 (VSS), A5.57 (VSS), A5.58 (VSS), C58.1, C62.1, U9.2 (GND)
- new net GND3: A5.2 (VDD), A5.3 (VDD), A5.4 (VDD), A5.41 (VDD), A5.42 (VDD), A5.49 (VDD), A5.5 (VDD), A5.50 (VDD), A5.51 (VDD), A5.52 (VDD), A5.59 (VDD), A5.6 (VDD), A5.60 (VDD), A5.7 (VDD), A5.8 (VDD), A8.14 (VSS), A8.21 (VSS), A8.22 (VSS), A8.23 (VSS), A8.24 (VSS), A8.25 (VSS), A8.26 (VSS), A8.27 (VSS), A8.28 (VSS), A8.35 (VSS), A8.36 (PINSEL), A8.43 (VSS), A8.44 (VSS), A8.45 (VSS), A8.46 (VSS), A8.47 (VSS), A8.48 (VSS), A8.53 (VSS), A8.54 (VSS), A8.55 (VSS), A8.56 (VSS), A8.57 (VSS), A8.58 (VSS), C49.2, C51.2, C57.1, C61.1, U8.2 (GND)
- new net REFCLKIN2: A5.29 (REFCLKIN)
- new net REFCLKOUT1: A1.38 (REFCLKOUT1)
- new net REFCLKOUT3: A5.38 (REFCLKOUT1)
- new net TRIP_1V2: A1.31 (TRIP_OUT), U7.6 (A4)
- new net Vcore: A8.2 (VDD), A8.3 (VDD), A8.4 (VDD), A8.41 (VDD), A8.42 (VDD), A8.49 (VDD), A8.5 (VDD), A8.50 (VDD), A8.51 (VDD), A8.52 (VDD), A8.59 (VDD), A8.6 (VDD), A8.60 (VDD), A8.7 (VDD), A8.8 (VDD)
- new net bypass1-1/out: A1.1 (VDD_INT_1)
- new net bypass1-2/in: A1.12 (VDD_INT_2)
- new net bypass4-1/out: A4.1 (VDD_INT_1)
- new net bypass4-2/in: A4.12 (VDD_INT_2)
- new net bypass5-1/out: A5.1 (VDD_INT_1)
- new net bypass5-2/in: A5.12 (VDD_INT_2)
- new net bypass8-1/out: A8.1 (VDD_INT_1)
- new net bypass8-2/in: A8.12 (VDD_INT_2)
- new net shifter2-3/RESET_IN: A4.17 (RESET_IN)
- new net shifter2-3/RESET_OUT: A1.16 (RESET_OUT)
- new net shifter2-3/RX_IN: A4.18 (RX_IN)
- new net shifter2-3/RX_OUT: A1.15 (RX_OUT)
- new net shifter2-3/TRIP_IN: A1.18 (TRIP_IN)
- new net shifter2-3/TRIP_OUT: A4.15 (TRIP_OUT)
- new net shifter2-3/TX_IN: A1.17 (TX_IN)
- new net shifter2-3/TX_OUT: A4.16 (TX_OUT)
- new net shifter4-5/RESET_IN: A5.33 (RESET_IN)
- new net shifter4-5/RESET_OUT: A4.32 (RESET_OUT)
- new net shifter4-5/RX_IN: A5.34 (RX_IN)
- new net shifter4-5/RX_OUT: A4.31 (RX_OUT)
- new net shifter4-5/TRIP_IN: A4.29 (REFCLKIN), A4.34 (TRIP_IN)
- new net shifter4-5/TRIP_OUT: A5.31 (TRIP_OUT)
- new net shifter4-5/TX_IN: A4.33 (TX_IN)
- new net shifter4-5/TX_OUT: A5.32 (TX_OUT)
- new net shifter6-7/RESET_IN: A8.17 (RESET_IN)
- new net shifter6-7/RESET_OUT: A5.16 (RESET_OUT)
- new net shifter6-7/RX_IN: A8.18 (RX_IN)
- new net shifter6-7/RX_OUT: A5.15 (RX_OUT)
- new net shifter6-7/TRIP_IN: A5.18 (TRIP_IN)
- new net shifter6-7/TRIP_OUT: A8.15 (TRIP_OUT)
- new net shifter6-7/TX_IN: A5.17 (TX_IN)
- new net shifter6-7/TX_OUT: A8.16 (TX_OUT)
- no-connect marks 5 -> 26
Other:
- added sheet bypass1-1 (bypass.kicad_sch)
- added sheet bypass1-2 (bypass.kicad_sch)
- added sheet bypass4-1 (bypass.kicad_sch)
- added sheet bypass4-2 (bypass.kicad_sch)
- added sheet bypass5-1 (bypass.kicad_sch)
- added sheet bypass5-2 (bypass.kicad_sch)
- added sheet bypass8-1 (bypass.kicad_sch)
- added sheet bypass8-2 (bypass.kicad_sch)
- added sheet shifter2-3 (shifter.kicad_sch)
- added sheet shifter4-5 (shifter.kicad_sch)
- added sheet shifter6-7 (shifter.kicad_sch)
- moved on the sheet: R28, TP14, TP22, U11, U6, U7

Commit message: finished adding ASICs to schematic. Change VR to single phase 2.8V output
Parts:
- removed C50: 120pF, Capacitor_SMD:C_0402_1005Metric, symbol Device:C_Small
- removed U6: 25MHz, bitaxe:SMD3225-4P, symbol bitaxe:oscillator
- added C62, C64: 120pF, Capacitor_SMD:C_0402_1005Metric, symbol Device:C_Small
- added Y2: 50MHz, bitaxe:OSC_ECS-3225MV-500-CN-TR, symbol bitaxe:oscillator
- TP15: renamed from TP19; value 1V2 -> 1V2-4
- TP16: renamed from TP20; value 1V2 -> 1V2-3
- TP17: renamed from TP21; value 1V2 -> 1V2-2
- TP18: renamed from TP22; value 1V2 -> 1V2-1
- renumbered A8 to A1, A5 to A2, A4 to A3, A1 to A4, C47 to C57, C46 to C58, C48 to C59, C49 to C60, C51 to C61, C52 to C63, C57 to C65, C58 to C66, C59 to C67, C60 to C68, C61 to C69, C62 to C70, C63 to C71, C64 to C72, R28 to R26, TP14 to TP10, TP15 to TP11, TP16 to TP12, TP17 to TP13, TP18 to TP14, U9 to U10, U10 to U11, U11 to U12, U7 to U8, U8 to U9
Connections:
- net CLKI is gone; now on net REFCLKIN1: A4.29 (REFCLKIN), TP10.1
- net bypass8-1/out is gone; now on net bypass4-1/out: A1.1 (VDD_INT_1)
- net bypass8-2/in is gone; now on net bypass4-2/in: A1.12 (VDD_INT_2)
- net shifter4-5/RESET_IN is gone; now on net shifter2-3/RESET_IN: A2.33 (RESET_IN)
- net shifter4-5/RESET_OUT is gone; now on net shifter2-3/RESET_OUT: A3.32 (RESET_OUT)
- net shifter4-5/RX_IN is gone; now on net shifter2-3/RX_IN: A2.34 (RX_IN)
- net shifter4-5/RX_OUT is gone; now on net shifter2-3/RX_OUT: A3.31 (RX_OUT)
- net shifter4-5/TRIP_OUT is gone; now on net shifter2-3/TRIP_OUT: A2.31 (TRIP_OUT)
- net shifter4-5/TX_IN is gone; now on net shifter2-3/TX_IN: A3.33 (TX_IN)
- net shifter4-5/TX_OUT is gone; now on net shifter2-3/TX_OUT: A2.32 (TX_OUT)
- net 1V2-1: now also A4.30 (VDDIO), C57.1, C58.1, C72.2, TP18.1, U12.5 (VOUT), U8.16 (VCCA), U8.2 (DIR2), U8.8 (DIR4), Y2.1 (EN), Y2.4 (VIN); no longer A3.30 (VDDIO), C71.2, TP17.1, U11.5 (VOUT)
- net 1V2-2: now also A3.30 (VDDIO), C71.2, TP17.1, U11.5 (VOUT); no longer A2.30 (VDDIO), C70.2, TP16.1, U10.5 (VOUT)
- net 1V2-3: now also A2.30 (VDDIO), C70.2, TP16.1, U10.5 (VOUT); no longer A1.30 (VDDIO), C69.2, TP15.1, U9.5 (VOUT)
- net GND: now also U8.7 (DIR3), C64.2, Y2.2 (GND); no longer U8.2 (DIR2)
- net GND2: now also C62.2
- net REFCLKIN1: now also Y2.3 (OUT)
- net REFCLKIN2: now also A3.29 (REFCLKIN); no longer A2.29 (REFCLKIN)
- net REFCLKIN3: now also A2.29 (REFCLKIN)
- net REFCLKOUT2: now also A3.38 (REFCLKOUT1)
- net bypass4-1/out: no longer A3.1 (VDD_INT_1)
- net bypass4-2/in: no longer A3.12 (VDD_INT_2)
- net shifter2-3/RESET_IN: no longer A3.17 (RESET_IN)
- net shifter2-3/RESET_OUT: no longer A4.16 (RESET_OUT)
- net shifter2-3/RX_IN: no longer A3.18 (RX_IN)
- net shifter2-3/RX_OUT: no longer A4.15 (RX_OUT)
- net shifter2-3/TRIP_IN: now also A3.34 (TRIP_IN); no longer A4.18 (TRIP_IN)
- net shifter2-3/TRIP_OUT: no longer A3.15 (TRIP_OUT)
- net shifter2-3/TX_IN: no longer A4.17 (TX_IN)
- net shifter2-3/TX_OUT: no longer A3.16 (TX_OUT)
- net at A2.20 (REFCLKOUT2): now also C62.1
- net REFCLKIN4: now reaches A1.29 (REFCLKIN)
- net at A4.20 (REFCLKOUT2): now also C64.1
- removed net 1V2: A4.30 (VDDIO), C57.1, C58.1, C72.2, TP18.1, U12.5 (VOUT), U8.16 (VCCA), U8.7 (DIR3), U8.8 (DIR4)
- net Vcore renamed VDD
- removed net shifter4-5/TRIP_IN: A3.29 (REFCLKIN), A3.34 (TRIP_IN)
- new net 1V2-4: A1.30 (VDDIO), C69.2, TP15.1, U9.5 (VOUT)
- new net bypass2-1/out: A3.1 (VDD_INT_1)
- new net bypass2-2/in: A3.12 (VDD_INT_2)
- new net shifter1-2/RESET_IN: A3.17 (RESET_IN)
- new net shifter1-2/RESET_OUT: A4.16 (RESET_OUT)
- new net shifter1-2/RX_IN: A3.18 (RX_IN)
- new net shifter1-2/RX_OUT: A4.15 (RX_OUT)
- new net shifter1-2/TRIP_IN: A4.18 (TRIP_IN)
- new net shifter1-2/TRIP_OUT: A3.15 (TRIP_OUT)
- new net shifter1-2/TX_IN: A4.17 (TX_IN)
- new net shifter1-2/TX_OUT: A3.16 (TX_OUT)
- no-connect marks 26 -> 30
Other:
- sheet bypass5-1 renamed bypass3-1
- sheet bypass5-2 renamed bypass3-2
- sheet shifter6-7 renamed shifter3-4
- removed sheet bypass8-1
- removed sheet bypass8-2
- removed sheet shifter4-5
- added sheet bypass2-1 (bypass.kicad_sch)
- added sheet bypass2-2 (bypass.kicad_sch)
- added sheet shifter1-2 (shifter.kicad_sch)
- sheet shifter2-3 ports: added GND_H, GND_L; removed GND0, GND1
- sheet shifter3-4 ports: added GND_H, GND_L; removed GND0, GND1
- moved on the sheet: A1, A2, A3, A4, C57, C58, C59, C60, C61, C63, C65, C66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

Commit message: switched to smaller level shifter diodes. switched ASIC modes
Parts:
- A1: renamed from A4; value BZM2_MODE1 -> BZM2_MODE0; symbol bitaxe:BZM2_mode1 -> bitaxe:BZM2_mode0
- A2: renamed from A3; value BZM2_MODE0 -> BZM2_MODE1; symbol bitaxe:BZM2_mode0 -> bitaxe:BZM2_mode1
- A3: renamed from A2; value BZM2_MODE1 -> BZM2_MODE0; symbol bitaxe:BZM2_mode1 -> bitaxe:BZM2_mode0
- A4: renamed from A1; value BZM2_MODE0 -> BZM2_MODE1; symbol bitaxe:BZM2_mode0 -> bitaxe:BZM2_mode1
- TP10: footprint TestPoint:TestPoint_Pad_D1.0mm -> bitaxe:TestPoint_Pad_D1.0mm
- TP11: value CLKI -> RX; footprint TestPoint:TestPoint_Pad_D1.0mm -> bitaxe:TestPoint_Pad_D1.0mm
- TP12: value CLKI -> RST; footprint TestPoint:TestPoint_Pad_D1.0mm -> bitaxe:TestPoint_Pad_D1.0mm
- TP13: value CLKI -> TX; footprint TestPoint:TestPoint_Pad_D1.0mm -> bitaxe:TestPoint_Pad_D1.0mm
- TP14: value CLKI -> TRP; footprint TestPoint:TestPoint_Pad_D1.0mm -> bitaxe:TestPoint_Pad_D1.0mm
- TP15, TP16, TP17, TP18: footprint TestPoint:TestPoint_Pad_D1.5mm -> bitaxe:TestPoint_Pad_D1.0mm
Connections:
- net GND: now also A1.36 (PINSEL)
- net GND1: no longer A2.36 (PINSEL)
- net GND2: now also A3.36 (PINSEL)
- net GND3: no longer A4.36 (PINSEL)
- net RST_1V2: now also A1.17 (RESET_IN); no longer A1.33 (RESET_IN)
- net RX_1V2: now also A1.18 (RX_IN); no longer A1.34 (RX_IN)
- net TRIP_1V2: now also A1.15 (TRIP_OUT); no longer A1.31 (TRIP_OUT)
- net TX_1V2: now also A1.16 (TX_OUT); no longer A1.32 (TX_OUT)
- net shifter1-2/RESET_IN: now also A2.32 (TX_OUT); no longer A2.17 (RESET_IN)
- net shifter1-2/RESET_OUT: now also A1.33 (TX_IN); no longer A1.16 (RESET_OUT)
- net shifter1-2/RX_IN: now also A2.31 (TRIP_OUT); no longer A2.18 (RX_IN)
- net shifter1-2/RX_OUT: now also A1.34 (TRIP_IN); no longer A1.15 (RX_OUT)
- net shifter1-2/TRIP_IN: now also A1.31 (RX_OUT); no longer A1.18 (TRIP_IN)
- net shifter1-2/TRIP_OUT: now also A2.34 (RX_IN); no longer A2.15 (TRIP_OUT)
- net shifter1-2/TX_IN: now also A1.32 (RESET_OUT); no longer A1.17 (TX_IN)
- net shifter1-2/TX_OUT: now also A2.33 (RESET_IN); no longer A2.16 (TX_OUT)
- net shifter2-3/RESET_IN: now also A3.17 (RESET_IN); no longer A3.33 (RESET_IN)
- net shifter2-3/RESET_OUT: now also A2.16 (RESET_OUT); no longer A2.32 (RESET_OUT)
- net shifter2-3/RX_IN: now also A3.18 (RX_IN); no longer A3.34 (RX_IN)
- net shifter2-3/RX_OUT: now also A2.15 (RX_OUT); no longer A2.31 (RX_OUT)
- net shifter2-3/TRIP_IN: now also A2.18 (TRIP_IN); no longer A2.34 (TRIP_IN)
- net shifter2-3/TRIP_OUT: now also A3.15 (TRIP_OUT); no longer A3.31 (TRIP_OUT)
- net shifter2-3/TX_IN: now also A2.17 (TX_IN); no longer A2.33 (TX_IN)
- net shifter2-3/TX_OUT: now also A3.16 (TX_OUT); no longer A3.32 (TX_OUT)
- net shifter3-4/RESET_IN: now also A4.33 (RESET_IN); no longer A4.17 (RESET_IN)
- net shifter3-4/RESET_OUT: now also A3.32 (RESET_OUT); no longer A3.16 (RESET_OUT)
- net shifter3-4/RX_IN: now also A4.34 (RX_IN); no longer A4.18 (RX_IN)
- net shifter3-4/RX_OUT: now also A3.31 (RX_OUT); no longer A3.15 (RX_OUT)
- net shifter3-4/TRIP_IN: now also A3.34 (TRIP_IN); no longer A3.18 (TRIP_IN)
- net shifter3-4/TRIP_OUT: now also A4.31 (TRIP_OUT); no longer A4.15 (TRIP_OUT)
- net shifter3-4/TX_IN: now also A3.33 (TX_IN); no longer A3.17 (TX_IN)
- net shifter3-4/TX_OUT: now also A4.32 (TX_OUT); no longer A4.16 (TX_OUT)
- net at TP14.1: now also A4.18 (TRIP_IN); no longer A4.34 (TRIP_IN)
- net at TP11.1: now also A4.15 (RX_OUT); no longer A4.31 (RX_OUT)
- net at TP12.1: now also A4.16 (RESET_OUT); no longer A4.32 (RESET_OUT)
- net at TP13.1: now also A4.17 (TX_IN); no longer A4.33 (TX_IN)
Other:
- moved on the sheet: C57, C59, C65, C66, C67, C68, C69, C70, C71, C72, R26, TP11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
