File: shifter.kicad_sch (KiCad schematic)
At the start: 11 parts

Commit message: cleaned up lots of ERC errors and warnings for #4
Changed lines of the file:
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@@
 		)
 	)
-	(label "GND1"
+	(label "GND_H"
 		(at 99.06 55.88 0)
 		(effects
