File: data.kicad_sch (KiCad schematic)
At the start: 17 parts, among them U5 TPS22919DCKR, U9 Raspberry Pi Pico

Commit message: power plane cleanup. added field vias. generated BOM
Parts:
- C45: LCSC C52923 -> (none)
- R20: LCSC C106235 -> (none)
Changed lines of the file:
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@@
 		(title "Bitaxe Intel Reference Design System")
 		(date "2025-10-01")
-		(rev "1300x")
+		(rev "1300xx")
 	)
 	(text "UART1"
@@
 			)
 		)
+		(property "Manufacturer" ""
+			(at 199.39 125.73 90)
+			(effects
+				(font
+					(size 1.27 1.27)
+				)
+				(hide yes)
+			)
+		)
 		(pin "1"
 		)
@@
 			)
 		)
+		(property "Manufacturer" ""
+			(at 246.38 123.19 90)
+			(effects
+				(font
+					(size 1.27 1.27)
+				)
+				(hide yes)
+			)
+		)
 		(pin "1"
 		)
@@
 			)
 		)
-		(property "LCSC" "C52923"
+		(property "LCSC" ""
 			(at 165.1 205.74 0)
 			(effects
@@
 		)
 		(property "Mouser" ""
+			(at 165.1 205.74 0)
+			(effects
+				(font
+					(size 1.27 1.27)
+				)
+				(hide yes)
+			)
+		)
+		(property "Manufacturer" ""
 			(at 165.1 205.74 0)
 			(effects
@@
 			)
 		)
+		(property "Manufacturer" ""
+			(at 186.69 204.47 0)
+			(effects
+				(font
+					(size 1.27 1.27)
+				)
+				(hide yes)
+			)
+		)
 		(pin "1"
 		)
@@
 			)
 		)
+		(property "Manufacturer" ""
+			(at 199.39 130.81 90)
+			(effects
+				(font
+					(size 1.27 1.27)
+				)
+				(hide yes)
+			)
+		)
 		(pin "1"
 		)
@@
 			)
 		)
+		(property "Manufacturer" ""
+			(at 248.92 105.41 90)
+			(effects
+				(font
+					(size 1.27 1.27)
+				)
+				(hide yes)
+			)
+		)
 		(pin "1"
 		)
@@
 		)
 		(property "Mouser" ""
+			(at 196.85 133.35 90)
+			(effects
+				(font
+					(size 1.27 1.27)
+				)
+				(hide yes)
+			)
+		)
+		(property "Manufacturer" ""
 			(at 196.85 133.35 90)
 			(effects
@@
 			)
 		)
-		(property "LCSC" "C106235"
+		(property "LCSC" ""
 			(at 200.66 201.93 0)
 			(effects
@@
 		)
 		(property "Mouser" ""
+			(at 200.66 201.93 0)
+			(effects
+				(font
+					(size 1.27 1.27)
+				)
+				(hide yes)
+			)
+		)
+		(property "Manufacturer" ""
 			(at 200.66 201.93 0)
 			(effects
@@
 			)
 		)
+		(property "Manufacturer" ""
+			(at 204.47 128.27 90)
+			(effects
+				(font
+					(size 1.27 1.27)
+				)
+				(hide yes)
+			)
+		)
 		(pin "1"
 		)
@@
 			)
 		)
+		(property "Manufacturer" ""
+			(at 176.53 140.97 90)
+			(effects
+				(font
+					(size 1.27 1.27)
+				)
+				(hide yes)
+			)
+		)
 		(pin "1"
 		)
@@
 			)
 		)
+		(property "Manufacturer" ""
+			(at 176.53 135.89 0)
+			(effects
+				(font
+					(size 1.27 1.27)
+				)
+				(hide yes)
+			)
+		)
 		(pin "1"
 		)
@@
 			)
 		)
+		(property "Manufacturer" ""
+			(at 170.18 140.97 90)
+			(effects
+				(font
+					(size 1.27 1.27)
+				)
+				(hide yes)
+			)
+		)
 		(pin "1"
 		)
@@
 			)
 		)
+		(property "Manufacturer" ""
+			(at 273.05 135.89 0)
+			(effects
+				(font
+					(size 1.27 1.27)
+				)
+				(hide yes)
+			)
+		)
 		(pin "1"
 		)
@@
 			)
 		)
+		(property "Manufacturer" ""
+			(at 170.18 135.89 0)
+			(effects
+				(font
+					(size 1.27 1.27)
+				)
+				(hide yes)
+			)
+		)
 		(pin "1"
 		)
@@
 		)
 		(property "Mouser" ""
+			(at 259.08 107.95 90)
+			(effects
+				(font
+					(size 1.27 1.27)
+				)
+				(hide yes)
+			)
+		)
+		(property "Manufacturer" ""
 			(at 259.08 107.95 90)
 			(effects
@@
 			)
 		)
+		(property "Manufacturer" ""
+			(at 226.06 121.92 0)
+			(effects
+				(font
+					(size 1.27 1.27)
+				)
+				(hide yes)
+			)
+		)
 		(pin "22"
 		)
@@
 			(at 196.85 123.19 90)
 			(effects
+				(font
+					(size 1.27 1.27)
+				)
+				(hide yes)
+			)
+		)
+		(property "Manufacturer" ""
+			(at 196.85 123.19 90)
+			(effects

Commit message: Correct U8 value field.
Parts:
- U9: value Raspberry Pi Pico -> Raspberry Pi Pico 2W
Changed lines of the file:
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@@
 		(on_board yes)
 		(dnp no)
-		(fields_autoplaced yes)
 		(property "Reference" "U9"
-			(at 226.06 88.9 0)
+			(at 215.138 91.948 0)
 			(effects
 				(font
@@
 			)
 		)
-		(property "Value" "Raspberry Pi Pico"
-			(at 226.06 91.44 0)
+		(property "Value" "Raspberry Pi Pico 2W"
+			(at 226.06 150.622 0)
 			(effects
 				(font

Commit message: cleaned up lots of ERC errors and warnings for #4
Connections:
- net TT_3V3 renamed TRIP_3V3
Changed lines of the file:
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@@
 		)
 	)
-	(hierarchical_label "TT_3V3"
+	(hierarchical_label "TRIP_3V3"
 		(shape input)
 		(at 195.58 130.81 180)
@@
 			)
 		)
-		(property "Description" ""
+		(property "Description" "test point"
 			(at 199.39 125.73 0)
 			(effects
@@
 			)
 		)
-		(property "Description" ""
+		(property "Description" "test point"
 			(at 246.38 123.19 0)
 			(effects
@@
 			)
 		)
-		(property "Description" ""
+		(property "Description" "test point"
 			(at 199.39 130.81 0)
 			(effects
@@
 			)
 		)
-		(property "Description" ""
+		(property "Description" "test point"
 			(at 248.92 105.41 0)
 			(effects
@@
 			)
 		)
-		(property "Description" ""
+		(property "Description" "test point"
 			(at 196.85 133.35 0)
 			(effects
@@
 			)
 		)
-		(property "Description" ""
+		(property "Description" "test point"
 			(at 204.47 128.27 0)
 			(effects
@@
 			)
 		)
-		(property "Description" ""
+		(property "Description" "test point"
 			(at 176.53 140.97 0)
 			(effects
@@
 			)
 		)
-		(property "Description" ""
+		(property "Description" "test point"
 			(at 170.18 140.97 0)
 			(effects
@@
 			)
 		)
-		(property "Description" ""
+		(property "Description" "test point"
 			(at 259.08 107.95 0)
 			(effects
@@
 			)
 		)
-		(property "Description" ""
+		(property "Description" "test point"
 			(at 196.85 123.19 0)
 			(effects
